File: rp2040_pad/rp2040_pad.kicad_pcb (KiCad board)
At the start: 2 copper layers, 71.3 x 86.1 mm, 58 parts, among them J1 USB_B_Micro, SW2 RotaryEncoder_Switch, SW3 RotaryEncoder_Switch, SW4 SW_Push, SW5 SW_Push, SW6 SW_Push, SW7 SW_Push, SW8 SW_Push, SW9 SW_Push, U1 RP2040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

Commit message: new design
Parts:
- removed C22: 0.1µ, Capacitor_SMD:C_1206_3216Metric
- removed G***: LOGO, LOGO
- removed RES1, USB_BOOT1: SW_Push, Button_Switch_THT:SW_PUSH_6mm
- added C20: 0.1µ, Capacitor_SMD:C_1206_3216Metric, F.Cu at (120.3, 102.8)
- added D13: LED, Inductor_SMD:L_1206_3216Metric, F.Cu at (118.0, 88.3)
- added D14: LED, Inductor_SMD:L_1206_3216Metric, F.Cu at (151.5, 89.3)
- added D15: LED, Inductor_SMD:L_1206_3216Metric, F.Cu at (140.9, 57.1)
- added R7: R, Resistor_SMD:R_1206_3216Metric, F.Cu at (118.0, 83.4)
- added R8: R, Resistor_SMD:R_1206_3216Metric, F.Cu at (146.2, 89.3)
- added R9: R, Resistor_SMD:R_1206_3216Metric, F.Cu at (135.7, 57.1)
- added RES: SW_Push, Button_Switch_THT:SW_PUSH_6mm, F.Cu at (133.1, 82.9)
- added USER_BOOT: SW_Push, Button_Switch_THT:SW_PUSH_6mm, F.Cu at (118.3, 58.0)
- H1, H2, H3, H4: footprint MountingHole:MountingHole_2.2mm_M2 -> MountingHole:MountingHole_3mm
- U3: footprint rp_2040_symbols:ABM8-272-T3 -> rp_2040_symbols:ABM8-272-T3-crystal
- moved H3 176.4 mm to (-7.33, 56.2)
- moved H2 166.8 mm to (-7.33, 50.2)
- moved H1 121.9 mm to (-7.33, 44.3)
- moved H4 101.5 mm to (-7.33, 62.1)
- moved R6 58.6 mm to (136.4, 90.3)
- moved D5 44.1 mm to (133.5, 106.7), turned to 0 degrees
- moved SW2 43.5 mm to (152.6, 102.5), turned to 180 degrees
- moved D12 41.0 mm to (117.0, 127.2)
- moved D11 39.7 mm to (133.0, 127.4)
- moved D1 39.1 mm to (97.0, 117.4)
- moved D6 39.0 mm to (96.7, 137.0)
- moved D2 38.9 mm to (117.0, 117.0)
- moved D3 38.9 mm to (136.8, 117.2)
- moved D7 38.4 mm to (116.7, 137.0)
- moved D8 38.4 mm to (136.5, 137.2)
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Connections:
- U1 pad 18: unconnected-(U1-GPIO15-Pad18) -> TEST_LED
- U1 pad 56: QSPI_SD1 -> QSPI_SS
Routing:
- net ENC_SA2: track 29.3 -> 77.3 mm, vias 2 -> 0
- net GND: track 75.8 -> 123.4 mm, vias 28 -> 53
- net ROW_B: track 75.2 -> 115.7 mm, vias 7 -> 6
- net ROW_A: track 106.9 -> 66.9 mm, vias 5 -> 3
- net ENC_SB2: track 39.9 -> 72.9 mm, vias 2 -> 0
- net ROW_C: track 92.6 -> 124.2 mm, vias 2 -> 8
- net Net-(U1-RUN): track 46.6 -> 22.2 mm, vias 3 -> 0
- net VBUS: track 140.2 -> 161.6 mm, vias 6 -> 13
- net COL_B: track 57.8 -> 74.9 mm
- net Net-(D10-DOUT): track 36.7 -> 20.1 mm, vias 4 -> 2
- net +3V3: track 161.8 -> 145.3 mm
- net QSPI_SD0: track 21.9 -> 7.40 mm
- net QSPI_SCLK: track 22.1 -> 8.97 mm
- net QSPI_SD3: track 23.4 -> 10.4 mm, vias 2 -> 0
- net QSPI_SS: track 10.1 -> 22.7 mm, vias 0 -> 2
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Other:
- board outline removed
- board text added: "3V3+"
- board text added: "P15"
- board text added: "TWIM"
- board text added: "VBUS"
- board text removed: "FIRST TRY?"
- board text removed: "RP_2040 MACRO PAD"

Commit message: added final version
Parts:
- added G***: LOGO, LOGO, F.Cu at (137.5, 62.8)
- added G***: LOGO, LOGO, B.Cu at (146.8, 66.0)
- added G***: LOGO, LOGO, B.Cu at (143.8, 142.5)
- C17, C18, C19, C20: footprint Capacitor_SMD:C_1206_3216Metric -> Capacitor_SMD:C_0805_2012Metric_Pad1.18x1.45mm_HandSolder
- moved H4 189.2 mm to (160.5, 149.5)
- moved H2 168.3 mm to (160.5, 62.5)
- moved H3 134.5 mm to (89.5, 149.5)
- moved H1 98.5 mm to (89.5, 62.5)
- moved R6 35.8 mm to (101.3, 83.0), turned to -90 degrees
- moved D15 29.8 mm to (152.7, 84.5), turned to 90 degrees
- moved RESET 29.1 mm to (104.1, 80.8)
- moved R9 28.0 mm to (152.8, 79.3), turned to -90 degrees
- moved D14 16.9 mm to (134.6, 90.2), turned to 0 degrees
- moved C1 7.53 mm to (144.9, 75.4)
- moved C10 7.53 mm to (131.8, 86.1)
- moved C11 7.53 mm to (131.9, 79.8)
- moved C12 7.53 mm to (137.1, 76.0)
- moved C13 7.53 mm to (137.1, 79.4)
- moved C14 7.53 mm to (137.1, 82.8)
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- renumbered RES to RESET, USER_BOOT to USB_BOOT1
Connections:
- U1 pad 11: COL_B -> ENC_SB2
- U1 pad 2: ENC_SA -> ROW_C
- U1 pad 3: ENC_SB -> ROW_B
- U1 pad 4: ENC_SA2 -> COL_A
- U1 pad 5: ENC_SB2 -> ROW_A
- U1 pad 6: ROW_A -> COL_B
- U1 pad 7: ROW_B -> ENC_SA
- U1 pad 8: ROW_C -> ENC_SB
- U1 pad 9: COL_A -> ENC_SA2
Routing:
- net VBUS: track 161.6 -> 213.0 mm, vias 13 -> 10
- net GND: track 123.4 -> 83.2 mm, vias 53 -> 37
- net ENC_SA2: track 77.3 -> 60.8 mm
- net ENC_SB2: track 72.9 -> 57.2 mm
- net COL_A: track 74.0 -> 87.3 mm, vias 2 -> 0
- net ROW_A: track 66.9 -> 54.6 mm, vias 3 -> 2
- net ROW_B: track 115.7 -> 126.3 mm
- net ENC_SA: track 38.5 -> 29.1 mm
- net LED: track 43.4 -> 34.4 mm
- net +3V3: track 145.3 -> 137.6 mm, vias 4 -> 41
- net ENC_SB: track 31.9 -> 24.3 mm
- net COL_C: track 86.8 -> 93.0 mm, vias 2 -> 1
- net Net-(U1-RUN): track 22.2 -> 27.9 mm, vias 0 -> 1
- net COL_B: track 74.9 -> 80.2 mm, vias 2 -> 0
- net ROW_C: track 124.2 -> 127.1 mm, vias 8 -> 0
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- added copper zone on B.Cu, net +3V3
- added copper zone on F.Cu, net +3V3
- added copper zone on F.Cu, net GND
Other:
- board outline added: 79 x 95 mm
- board text added: "SECOND TRY ?"
- board text removed: "TWIM"
