File: rp2040_pad/rp2040_pad.kicad_sch (KiCad schematic)
At the start: 57 parts, among them J1 USB_B_Micro, SW2 RotaryEncoder_Switch, SW3 RotaryEncoder_Switch, SW4 SW_Push, SW5 SW_Push, SW6 SW_Push, SW7 SW_Push, SW8 SW_Push, SW9 SW_Push, U1 RP2040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

Commit message: new design
Parts:
- added D13, D14, D15: LED, Inductor_SMD:L_1206_3216Metric, symbol Device:LED
- added R7, R8, R9: R, Resistor_SMD:R_1206_3216Metric, symbol Device:R
- H1, H2, H3, H4: footprint MountingHole:MountingHole_2.2mm_M2 -> MountingHole:MountingHole_3mm
- U3: footprint rp_2040_symbols:ABM8-272-T3 -> rp_2040_symbols:ABM8-272-T3-crystal
Connections:
- net +3V3: now also R8.1
- net GND: now also D13.1 (K), D14.1 (K), D15.1 (K)
- net QSPI_SD1: no longer U1.56 (QSPI_SS)
- net QSPI_SS: now also U1.56 (QSPI_SS)
- net VBUS: now also R9.1
- net TEST_LED: now reaches U1.18 (GPIO15)
- net TEST_LED: now also R7.1
- new net: D13.2 (A), R7.2
- new net: D15.2 (A), R9.2
- new net: D14.2 (A), R8.2
- no-connect marks 23 -> 22
Other:
- note added: "TEST LEDS"

Commit message: added final version
Parts:
- C17, C18, C19, C20: footprint Capacitor_SMD:C_1206_3216Metric -> Capacitor_SMD:C_0805_2012Metric_Pad1.18x1.45mm_HandSolder
Connections:
- net COL_A: now also U1.4 (GPIO2); no longer U1.9 (GPIO7)
- net COL_B: now also U1.6 (GPIO4); no longer U1.11 (GPIO8)
- net ENC_SA: now also U1.7 (GPIO5); no longer U1.2 (GPIO0)
- net ENC_SA2: now also U1.9 (GPIO7); no longer U1.4 (GPIO2)
- net ENC_SB: now also U1.8 (GPIO6); no longer U1.3 (GPIO1)
- net ENC_SB2: now also U1.11 (GPIO8); no longer U1.5 (GPIO3)
- net ROW_A: now also U1.5 (GPIO3); no longer U1.6 (GPIO4)
- net ROW_B: now also U1.3 (GPIO1); no longer U1.7 (GPIO5)
- net ROW_C: now also U1.2 (GPIO0); no longer U1.8 (GPIO6)
